Commit message: chore: Update file paths and include new manipulator component in vera.urdf.xacro

File: urdf/mech/base.urdf.xacro (robot description, xacro)
@@ -43,6 +43,6 @@
     </joint>
   </xacro:macro>
-  <xacro:macro name="torso" params="length width height mass pos_z pos_x">
-    <link name="torso">
+  <xacro:macro name="torso_link" params="length width height mass pos_z pos_x">
+    <link name="torso_link">
       <visual>
         <origin xyz="${-length/2 - 0.015} 0 ${-height/2}" rpy="1.57 0 0"/>
@@ -70,5 +70,5 @@
     <joint name="base_to_torso" type="fixed">
       <parent link="base_link"/>
-      <child link="torso"/>
+      <child link="torso_link"/>
       <origin xyz="${pos_x} 0 ${pos_z}" rpy="0 0 0"/>
     </joint>

File: urdf/robots/vera.urdf.xacro (robot description, xacro)
@@ -1,5 +1,5 @@
 <?xml version="1.0"?>
 <robot name="linorobot2_2wd" xmlns:xacro="http://ros.org/wiki/xacro">
-  <xacro:include filename="$(find vera_description)/urdf/mecanum_properties.urdf.xacro" />
+  <xacro:include filename="$(find vera_description)/urdf/utils/mecanum_properties.urdf.xacro" />
   <xacro:include filename="$(find vera_description)/urdf/mech/base.urdf.xacro" />
   <xacro:include filename="$(find vera_description)/urdf/mech/mecanum_wheel.urdf.xacro" />
@@ -8,4 +8,5 @@
   <xacro:include filename="$(find vera_description)/urdf/sensors/depth_sensor.urdf.xacro" />
   <xacro:include filename="$(find vera_description)/urdf/controllers/omni_drive.urdf.xacro" />
+  <xacro:include filename="$(find vera_description)/urdf/mech/manipulator.xml" />
   <xacro:base
     length="${base_length}"
@@ -51,5 +52,5 @@
     mass="${wheel_mass}"
   />
-  <xacro:torso
+  <xacro:torso_link
     length="${torso_length}"
     width="${torso_width}"
@@ -59,4 +60,5 @@
     pos_x="${torso_pos_x}"
   />
+  <xacro:manipulator/>
   <!-- <xacro:imu/>
   <xacro:generic_laser>

Commit message: chore: Update file paths and include new manipulator component in vera.urdf.xacro

File: urdf/mech/base.urdf.xacro (robot description, xacro)
@@ -7,5 +7,5 @@
         <origin xyz="${-length/2} ${-width/2} ${-height/2}" rpy="1.57 0 0"/>
         <geometry>
-          <mesh filename="package://vera_description/meshes/structure/base.stl" scale="0.001 0.001 0.001"/>
+          <mesh filename="file://$(find vera_description)/meshes/structure/base.stl" scale="0.001 0.001 0.001"/>
         </geometry>
         <material name="yellow">
@@ -14,7 +14,7 @@
       </visual>
       <collision>
-        <origin xyz="0 0 0" rpy="0 0 0"/>
+        <origin xyz="${-length/2} ${-width/2} ${-height/2}" rpy="1.57 0 0"/>
         <geometry>
-          <box size="${length} ${width} ${height}"/>
+          <mesh filename="file://$(find vera_description)/meshes/structure/base.stl" scale="0.001 0.001 0.001"/>
         </geometry>
       </collision>
@@ -48,5 +48,5 @@
         <origin xyz="${-length/2 - 0.015} 0 ${-height/2}" rpy="1.57 0 0"/>
         <geometry>
-          <mesh filename="package://vera_description/meshes/structure/torso.stl" scale="0.001 0.001 0.001"/>
+          <mesh filename="file://$(find vera_description)/meshes/structure/torso.stl" scale="0.001 0.001 0.001"/>
         </geometry>
         <material name="yellow">
@@ -57,5 +57,5 @@
         <origin xyz="${-length/2 - 0.015} 0 ${-height/2}" rpy="1.57 0 0"/>
         <geometry>
-          <box size="${length} ${width} ${height}"/>
+          <mesh filename="file://$(find vera_description)/meshes/structure/torso.stl" scale="0.001 0.001 0.001"/>
         </geometry>
       </collision>

File: urdf/robots/vera.urdf.xacro (robot description, xacro)
@@ -1,4 +1,4 @@
 <?xml version="1.0"?>
-<robot name="linorobot2_2wd" xmlns:xacro="http://ros.org/wiki/xacro">
+<robot name="vera" xmlns:xacro="http://ros.org/wiki/xacro">
   <xacro:include filename="$(find vera_description)/urdf/utils/mecanum_properties.urdf.xacro" />
   <xacro:include filename="$(find vera_description)/urdf/mech/base.urdf.xacro" />
